File: HM-PWR-WTH-2/HM-PWR-WTH-2.kicad_pcb (KiCad board)
At the start: 2 copper layers, 45 x 43 mm, 42 parts, among them J101 Screw_Terminal_01x02, J102 Conn_01x02_Male, J103 Conn_01x02_Male, J104 Conn_01x02_Male, J105 Conn_01x02_Male, J106 USB_B_Micro, SW101 SW_Push, SW102 SW_Push, U101 LT8606xMSE

Commit message: HM-PWR-WTH-2: Finalize the layout
Signed-off-by: Patrick Rudolph <siro@das-labor.org>
Parts:
- J106: footprint Connector_USB:USB_Micro-B_GCT_USB3076-30-A -> Connector_USB:USB_Micro-B_Amphenol_10104110_Horizontal
- moved J106 10.6 mm to (103.5, 83.0)
- moved C117 9.82 mm to (98.0, 96.8), turned to 270 degrees
- moved C108 5.54 mm to (101.0, 96.7), turned to 90 degrees
- moved J101 3.68 mm to (90.2, 87.0)
- moved D103 1.88 mm to (82.3, 95.0), turned to 180 degrees
- moved R108 1.41 mm to (78.5, 97.0), turned to 270 degrees
- moved SW102 1.35 mm to (83.8, 84.2)
- turned C110 to 0 degrees
- turned C111 to 0 degrees
- turned C113 to 0 degrees
- turned C118 to 180 degrees
Routing:
- net 3V0: track 118.1 -> 94.9 mm, vias 4 -> 8
- net Net-(D101-Pad2): track 6.20 -> 10.1 mm
- net Net-(D104-Pad2): track 6.66 -> 8.35 mm
- net GND: track 1.28 -> 2.91 mm, vias 44 -> 41
- net Net-(D103-Pad1): track 9.75 -> 10.8 mm
- net Net-(C101-Pad2): track 8.56 -> 9.52 mm
- net +24V: track 8.86 -> 9.54 mm
- added copper zone on F.Cu, net 3V0
