File: HM-PWR-WTH-2/HM-PWR-WTH-2.sch (KiCad schematic (older format))
At the start: 42 parts, among them J101 Screw_Terminal_01x02, J102 Conn_01x02_Male, J103 Conn_01x02_Male, J104 Conn_01x02_Male, J105 Conn_01x02_Male, J106 USB_B_Micro, SW101 SW_Push, SW102 SW_Push, U101 LT8606xMSE

Commit message: HM-PWR-WTH-2: Finalize the layout
Signed-off-by: Patrick Rudolph <siro@das-labor.org>
Parts:
- J106: footprint Connector_USB:USB_Micro-B_GCT_USB3076-30-A -> Connector_USB:USB_Micro-B_Amphenol_10104110_Horizontal
Changed lines of the file:
@@
 F 0 "J106" H 2107 6517 50  0000 C CNN
 F 1 "USB_B_Micro" H 2107 6426 50  0000 C CNN
-F 2 "Connector_USB:USB_Micro-B_GCT_USB3076-30-A" H 2200 6000 50  0001 C CNN
+F 2 "Connector_USB:USB_Micro-B_Amphenol_10104110_Horizontal" H 2200 6000 50  0001 C CNN
 F 3 "~" H 2200 6000 50  0001 C CNN
 	1    2050 6050
